File: Lab4/ExerciseI/Lab6/Lab6.kicad_sch (KiCad schematic)
At the start: 6 parts, among them SW1 SW_SPDT

Commit message: Lab 6 PCB Designs
Parts:
- R1: value 20 kΩ -> 2.2 kΩ
- R2: value 2.2 kΩ -> 20 kΩ
Connections:
- net at R2.1: now also D1.2 (A); no longer V1.1 (Pin_1)
- net at R1.1: now also V1.1 (Pin_1); no longer D1.2 (A)
- net at R2.2: now also C1.1, SW1.3 (C); no longer SW1.2 (B)
- new net: R1.2, SW1.2 (B)
