File: Lab4/Lab6II/555Timer/_autosave-555Timer.kicad_sch (KiCad schematic)
At the start: 10 parts, among them U1 U1

Commit message: Lab 6 PCB Designs
Parts:
- removed +9V: Conn_01x02_Male, TerminalBlock:TerminalBlock_bornier-2_P5.08mm, symbol Connector:Conn_01x02_Male
- added +9V1: Conn_01x02_Male, TerminalBlock:TerminalBlock_bornier-2_P5.08mm, symbol Connector:Conn_01x02_Male
- D2: footprint (none) -> LED_SMD:LED_1206_3216Metric_Pad1.42x1.75mm_HandSolder
Connections:
- net +9V: now also +9V1.1 (Pin_1)
- net GND: now also +9V1.2 (Pin_2)
Other:
- note removed: "2023 - 01 - 27"
- note removed: "555 Timer Circuit"
