File: Lab4/Lab6II/555Timer/555Timer.kicad_pcb (KiCad board)
At the start: 2 copper layers, 46.3 x 35.5 mm, 10 parts, among them U1 U1

Commit message: Lab #6 Final
Routing:
- net /pin_2: track 35.1 -> 58.3 mm, vias 0 -> 2
- net /pin_3: track 20.2 -> 38.5 mm, vias 2 -> 3
- net +9V: track 53.5 -> 67.5 mm, vias 0 -> 2

Commit message: Lab 7 Gerber and Drill Files
Parts:
- moved R4 2.18 mm to (221.5, 142.9)
Routing:
- net /pin_3: track 38.5 -> 42.1 mm
- net Net-(R4-Pad2): track 14.7 -> 17.2 mm
- net /pin_2: track 58.3 -> 59.3 mm
- added copper zone on B.Cu, net GND
- added copper zone on F.Cu, net GND
Other:
- outline, holes or cut-outs redrawn
Changed lines of the file:
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@@
       (sketchpadsonfab false)
       (subtractmaskfromsilk false)
-      (outputformat 4)
+      (outputformat 1)
       (mirror false)
       (drillshape 0)
       (scaleselection 1)
-      (outputdirectory "./")
+      (outputdirectory "../../../Lab7Gerbers/")
     )
   )
@@
     (property "Sheetname" "")
     (attr smd)
-    (fp_text reference "R1" (at 0 -1.65 90) (layer "F.SilkS")
-      (effects (font (size 1 1) (thickness 0.15)))
-    )
-    (fp_text value "1k" (at 0 1.65 90) (layer "F.Fab")
+    (fp_text reference "R1" (at 0.1684 1.7272 90) (layer "F.SilkS")
+      (effects (font (size 1 1) (thickness 0.15)))
+    )
+    (fp_text value "1k" (at 0.3716 -1.6764 90) (layer "F.Fab")
       (effects (font (size 1 1) (thickness 0.15)))
     )
@@
     (property "Sheetname" "")
     (attr smd)
-    (fp_text reference "D1" (at 0 -1.82 90) (layer "F.SilkS")
-      (effects (font (size 1 1) (thickness 0.15)))
-    )
-    (fp_text value "LED" (at 0 1.82 90) (layer "F.Fab")
+    (fp_text reference "D1" (at -0.3302 1.8685 90) (layer "F.SilkS")
+      (effects (font (size 1 1) (thickness 0.15)))
+    )
+    (fp_text value "LED" (at -0.1778 -1.9923 90) (layer "F.Fab")
       (effects (font (size 1 1) (thickness 0.15)))
     )
@@
   )
   (footprint "Resistor_SMD:R_0805_2012Metric_Pad1.20x1.40mm_HandSolder" (layer "F.Cu")
-    (at 223.3168 141.6464 -90)
+    (at 221.5134 142.875 -90)
     (descr "Resistor SMD 0805 (2012 Metric), square (rectangular) end terminal, IPC_7351 nominal with elongated pad for handsoldering. (Body size source: IPC-SM-782 page 72, https://www.pcb-3d.com/wordpress/wp-content/uploads/ipc-sm-782a_amendment_1_and_2.pdf), generated with kicad-footprint-generator")
     (tags "resistor handsolder")
@@
       (effects (font (size 1 1) (thickness 0.15)))
     )
-    (fp_text value "Conn_01x02_Male" (at 2.54 5.08) (layer "F.Fab")
+    (fp_text value "Conn_01x02_Male" (at -9.8298 -2.9972) (layer "F.Fab")
       (effects (font (size 1 1) (thickness 0.15)))
     )
@@
     )
   )
-  (gr_circle (center 200.6092 113.6142) (end 201.957316 113.6142) (layer "Edge.Cuts") (width 0.1) (fill none))
+  (gr_circle (center 201.1172 113.9444) (end 202.465316 113.9444) (layer "Edge.Cuts") (width 0.1) (fill none))
   (gr_rect (start 198.7042 111.5822) (end 244.983 147.0914) (layer "Edge.Cuts") (width 0.1) (fill none))
   (gr_text "Vega PCB" (at 240.5634 145.4404) (layer "F.SilkS")
     (effects (font (size 1 1) (thickness 0.15)))
   )
-  (gr_text "555 Timer" (at 206.629 113.7666) (layer "F.SilkS")
+  (gr_text "555 Timer" (at 206.9338 113.5126) (layer "F.SilkS")
     (effects (font (size 1 1) (thickness 0.15)))
   )
@@
   (via (at 223.7486 128.4732) (size 0.8) (drill 0.4) (layers "F.Cu" "B.Cu") (net 4))
   (via (at 229.0318 136.2202) (size 0.8) (drill 0.4) (layers "F.Cu" "B.Cu") (net 4))
-  (segment (start 229.0318 136.2202) (end 229.0318 133.7564) (width 0.254) (layer "B.Cu") (net 4))
-  (segment (start 229.0318 133.7564) (end 223.7486 128.4732) (width 0.254) (layer "B.Cu") (net 4))
+  (segment (start 225.552 128.4732) (end 223.7486 128.4732) (width 0.254) (layer "B.Cu") (net 4))
+  (segment (start 229.0318 131.953) (end 225.552 128.4732) (width 0.254) (layer "B.Cu") (net 4))
+  (segment (start 229.0318 136.2202) (end 229.0318 131.953) (width 0.254) (layer "B.Cu") (net 4))
   (segment (start 238.8473 123.7377) (end 238.4298 124.1552) (width 0.254) (layer "F.Cu") (net 5))
   (segment (start 238.4298 124.1552) (end 238.4298 128.8288) (width 0.254) (layer "F.Cu") (net 5))
@@
   (segment (start 216.4842 139.0142) (end 224.6884 139.0142) (width 0.254) (layer "B.Cu") (net 6))
   (segment (start 216.2556 134.366) (end 216.2556 138.7856) (width 0.254) (layer "B.Cu") (net 6))
-  (segment (start 226.6884 140.6464) (end 227.965 139.3698) (width 0.254) (layer "F.Cu") (net 7))
   (segment (start 234.855 127.254) (end 238.4298 130.8288) (width 0.254) (layer "F.Cu") (net 7))
   (segment (start 229.235 127.254) (end 234.855 127.254) (width 0.254) (layer "F.Cu") (net 7))
+  (segment (start 227.965 139.3698) (end 225.4598 141.875) (width 0.254) (layer "F.Cu") (net 7))
   (segment (start 222.4398 128.385) (end 223.5708 127.254) (width 0.254) (layer "F.Cu") (net 7))
   (segment (start 222.4398 130.683) (end 222.4398 128.385) (width 0.254) (layer "F.Cu") (net 7))
-  (segment (start 223.3168 140.6464) (end 226.6884 140.6464) (width 0.254) (layer "F.Cu") (net 7))
+  (segment (start 225.4598 141.875) (end 221.5134 141.875) (width 0.254) (layer "F.Cu") (net 7))
   (via (at 223.5708 127.254) (size 0.8) (drill 0.4) (layers "F.Cu" "B.Cu") (net 7))
   (via (at 227.965 139.3698) (size 0.8) (drill 0.4) (layers "F.Cu" "B.Cu") (net 7))
   (via (at 229.235 127.254) (size 0.8) (drill 0.4) (layers "F.Cu" "B.Cu") (net 7))
-  (segment (start 227.965 139.3698) (end 229.7588 137.576) (width 0.254) (layer "B.Cu") (net 7))
   (segment (start 223.5708 127.254) (end 229.235 127.254) (width 0.254) (layer "B.Cu") (net 7))
-  (segment (start 229.7588 127.7778) (end 229.235 127.254) (width 0.254) (layer "B.Cu") (net 7))
-  (segment (start 229.7588 137.576) (end 229.7588 127.7778) (width 0.254) (layer "B.Cu") (net 7))
-  (segment (start 224.7106 141.2526) (end 223.3168 142.6464) (width 0.254) (layer "F.Cu") (net 8))
-  (segment (start 237.4392 141.2526) (end 224.7106 141.2526) (width 0.254) (layer "F.Cu") (net 8))
+  (segment (start 227.965 139.3698) (end 231.3686 135.9662) (width 0.254) (layer "B.Cu") (net 7))
+  (segment (start 231.3686 129.3876) (end 229.235 127.254) (width 0.254) (layer "B.Cu") (net 7))
+  (segment (start 231.3686 135.9662) (end 231.3686 129.3876) (width 0.254) (layer "B.Cu") (net 7))
+  (segment (start 234.5976 144.0942) (end 221.7326 144.0942) (width 0.254) (layer "F.Cu") (net 8))
+  (segment (start 237.4392 141.2526) (end 234.5976 144.0942) (width 0.254) (layer "F.Cu") (net 8))
+  (segment (start 221.7326 144.0942) (end 221.5134 143.875) (width 0.254) (layer "F.Cu") (net 8))
+  (zone (net 2) (net_name "GND") (layer "F.Cu") (hatch edge 0.508)
+    (connect_pads (clearance 0.508))
+    (min_thickness 0.254) (filled_areas_thickness no)
+    (fill yes (thermal_gap 0.508) (thermal_bridge_width 0.508))
+    (polygon
+      (pts
+        (xy 245.2116 111.3282)
+        (xy 245.2116 147.3454)
+        (xy 198.501 147.3962)
+        (xy 198.3486 147.3962)
+        (xy 198.3994 111.2266)
+      )
+    )
+  )
+  (zone (net 2) (net_name "GND") (layer "B.Cu") (hatch edge 0.508)
+    (connect_pads (clearance 0.508))
+    (min_thickness 0.254) (filled_areas_thickness no)
+    (fill yes (thermal_gap 0.508) (thermal_bridge_width 0.508))
+    (polygon
+      (pts
+        (xy 245.2116 147.4978)
+        (xy 198.4502 147.3962)
+        (xy 198.247 111.4298)
+        (xy 245.3894 111.2266)
+      )
+    )
+  )
 )
