File: Lab4/Lab6II/555Timer/555Timer.kicad_sch (KiCad schematic)
At the start: 10 parts, among them U1 U1

Commit message: Lab 6 PCB Designs
Parts:
- removed +9V: Conn_01x02_Male, TerminalBlock:TerminalBlock_bornier-2_P5.08mm, symbol Connector:Conn_01x02_Male
- added +9V1: Conn_01x02_Male, TerminalBlock:TerminalBlock_bornier-2_P5.08mm, symbol Connector:Conn_01x02_Male
Connections:
- net +9V: now also +9V1.1 (Pin_1)
- net GND: now also +9V1.2 (Pin_2)
Other:
- note removed: "2023 - 01 - 27"
- note removed: "555 Timer Circuit"

Commit message: Lab 7 Gerber and Drill Files
Parts:
- D2: footprint (none) -> LED_SMD:LED_1206_3216Metric_Pad1.42x1.75mm_HandSolder
Changed lines of the file:
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@@
       (effects (font (size 1.27 1.27)) (justify right))
     )
-    (property "Footprint" "" (id 2) (at 265.43 142.24 0)
+    (property "Footprint" "LED_SMD:LED_1206_3216Metric_Pad1.42x1.75mm_HandSolder" (id 2) (at 265.43 142.24 0)
       (effects (font (size 1.27 1.27)) hide)
     )
@@
     )
     (path "/f85b65f6-7a19-460e-acd9-046d91c128fd"
-      (reference "D2") (unit 1) (value "LED") (footprint "")
+      (reference "D2") (unit 1) (value "LED") (footprint "LED_SMD:LED_1206_3216Metric_Pad1.42x1.75mm_HandSolder")
     )
     (path "/4ef93625-99f1-41f4-a186-dc77b7dc091e"
